Commit message: add new model robot docking

File: robot_da/src/robot_docking/urdf/robot_docking.urdf.xacro (robot description, xacro)
@@ -6,4 +6,10 @@
   <xacro:include filename="$(find robot_docking)/urdf/robot_properties.xacro" />
   <xacro:include filename="$(find robot_docking)/urdf/common_properties.xacro" />
+  <xacro:property name="base_edge" value="0.13"/>
+  <xacro:property name="base_mass" value="0.033"/>
+  <xacro:property name="base_pos" value="0.02"/>
+  <xacro:property name="wheel_radius" value="0.02"/>
+  <xacro:property name="wheel_length" value="0.02"/>
+  <xacro:property name="wheel_mass" value="0.006"/>
   <link name="basefoot_link" />
   <link
@@ -11,15 +17,15 @@
     <inertial>
       <origin
-        xyz="0.000289864579681387 -0.000718230891326076 0.047950882279495"
-        rpy="0 0 0" />
-      <mass
-        value="0.331171188980549" />
-      <inertia
-        ixx="0.00111418343424523"
-        ixy="-5.44568062251066E-06"
-        ixz="-2.02304877726191E-06"
-        iyy="0.00110250630250282"
-        iyz="2.54448430715081E-06"
-        izz="0.0014284323191472" />
+        xyz="0.000299996753193699 -0.000738676101724914 0.0493158011467332"
+        rpy="0 0 0" />
+      <mass
+        value="0.319986271762139" />
+      <inertia
+        ixx="0.00111389760044166"
+        ixy="-5.44568054171093E-06"
+        ixz="-2.02304849683939E-06"
+        iyy="0.00110222046873689"
+        iyz="2.54448439440798E-06"
+        izz="0.00142810340911259" />
     </inertial>
     <visual>
@@ -39,5 +45,5 @@
     <collision>
       <origin
-        xyz="0 0 0.02"
+        xyz="0 0 0"
         rpy="0 0 0" />
       <geometry>
@@ -56,15 +62,15 @@
     <inertial>
       <origin
-        xyz="-0.00324040376374836 4.89031228385201E-06 1.42076747643854E-06"
-        rpy="0 0 0" />
-      <mass
-        value="0.00618073560320388" />
-      <inertia
-        ixx="5.71253232809819E-07"
-        ixy="-1.0358180535669E-13"
-        ixz="-4.14569771104536E-14"
-        iyy="2.94198592880854E-07"
-        iyz="2.98405896563239E-10"
-        izz="2.93572446838264E-07" />
+        xyz="-0.000185240624970454 8.47068578512453E-05 1.75601486899143E-05"
+        rpy="0 0 0" />
+      <mass
+        value="0.00691755480566768" />
+      <inertia
+        ixx="5.82243996732172E-07"
+        ixy="-1.17470086109394E-14"
+        ixz="1.14622550432559E-13"
+        iyy="3.07378635100047E-07"
+        iyz="-7.08882546315987E-11"
+        izz="3.03751087072827E-07" />
     </inertial>
     <visual>
@@ -96,5 +102,5 @@
     type="continuous">
     <origin
-      xyz="0.0466666666666667 -0.00020526372785272 0.00799951222526741"
+      xyz="0.0433333333333333 -0.00020000000000002 0.00799999999999999"
       rpy="0 0 0" />
     <parent
@@ -103,5 +109,5 @@
       link="front_wheel_link" />
     <axis
-      xyz="-1 0 0" />
+      xyz="1 0 0" />
     <limit
       effort="0.38195"
@@ -115,15 +121,15 @@
     <inertial>
       <origin
-        xyz="0.00161977052337231 -0.00280652102287197 5.06810032584182E-06"
-        rpy="0 0 0" />
-      <mass
-        value="0.00618073560320388" />
-      <inertia
-        ixx="3.62903069155732E-07"
-        ixy="-1.2029102307139E-07"
-        ixz="5.57850139767036E-14"
-        iyy="5.01803178258457E-07"
-        iyz="-9.66224794778852E-14"
-        izz="2.94318025114749E-07" />
+        xyz="1.88093972769421E-05 -0.000203080237360819 -1.45462319701764E-05"
+        rpy="0 0 0" />
+      <mass
+        value="0.00691755480566768" />
+      <inertia
+        ixx="3.75694147764389E-07"
+        ixy="-1.19251631263871E-07"
+        ixz="1.11530814759738E-09"
+        iyy="5.13394034485272E-07"
+        iyz="6.43973090634511E-10"
+        izz="3.04285419017751E-07" />
     </inertial>
     <visual>
@@ -155,5 +161,5 @@
     type="continuous">
     <origin
-      xyz="-0.0235052367476054 0.0403152703607692 0.00799493189967413"
+      xyz="-0.0218398717474237 0.0374277674973255 0.00799999999999983"
       rpy="0 0 0" />
     <parent
@@ -162,5 +168,5 @@
       link="left_wheel_link" />
     <axis
-      xyz="0.500000000000001 -0.866025403784438 0" />
+      xyz="-0.500000000000002 0.866025403784437 0" />
     <limit
       effort="0.38195"
@@ -174,15 +180,15 @@
     <inertial>
       <origin
-        xyz="0.00171747127062813 0.00296472511820606 9.06473329523316E-07"
-        rpy="0 0 0" />
-      <mass
-        value="0.00618073560320387" />
-      <inertia
-        ixx="3.63503429118346E-07"
-        ixy="1.19944512404821E-07"
-        ixz="1.97017670949224E-10"
-        iyy="5.02003174324161E-07"
-        iyz="-1.13712984044728E-10"
-        izz="2.93517669086433E-07" />
+        xyz="0.000166197887385422 0.00011801735843614 1.69662306176849E-05"
+        rpy="0 0 0" />
+      <mass
+        value="0.00691755480566768" />
+      <inertia
+        ixx="3.76094071379335E-07"
+        ixy="1.19020850771271E-07"
+        ixz="-8.64105503461082E-11"
+        iyy="5.13527647804894E-07"
+        iyz="4.98035582698257E-11"
+        izz="3.03752422351457E-07" />
     </inertial>
     <visual>
@@ -214,5 +220,5 @@
     type="continuous">
     <origin
-      xyz="-0.0231647060085328 -0.0405118758746402 0.0080000601855697"
+      xyz="-0.0214934615859098 -0.0376277674973257 0.008"
       rpy="0 0 0" />
     <parent
@@ -221,5 +227,5 @@
       link="right_wheel_link" />
     <axis
-      xyz="0.500000000000001 0.866025403784438 0" />
+      xyz="-0.5 -0.866025403784438 0" />
     <limit
       effort="0.38195"
@@ -233,5 +239,5 @@
     <inertial>
       <origin
-        xyz="-5.55111512312578E-17 2.77555756156289E-17 -0.0025"
+        xyz="-1.11022302462516E-16 1.2490009027033E-16 -0.00250000000000001"
         rpy="0 0 0" />
       <mass
@@ -239,8 +245,8 @@
       <inertia
         ixx="2.80265403074513E-07"
-        ixy="-5.9557004103818E-23"
-        ixz="5.29395592033938E-23"
-        iyy="2.80265403074513E-07"
-        iyz="-2.16721320488893E-22"
+        ixy="-8.27180612553028E-25"
+        ixz="1.05879118406788E-22"
+        iyy="2.80265403074512E-07"
+        iyz="-2.41536738865484E-22"
         izz="5.05950422035626E-07" />
     </inertial>
@@ -298,8 +304,8 @@
       <inertia
         ixx="4.08944526124647E-06"
-        ixy="4.10281583826302E-22"
-        ixz="0"
+        ixy="-3.30872245021211E-22"
+        ixz="-1.05879118406788E-22"
         iyy="4.08944526124647E-06"
-        iyz="-7.94093388050907E-23"
+        iyz="-3.97046694025453E-22"
         izz="8.02453487611104E-06" />
     </inertial>
@@ -357,8 +363,8 @@
       <inertia
         ixx="7.00800168489498E-07"
-        ixy="-7.09565236577912E-15"
-        ixz="-7.90343014493252E-08"
+        ixy="-7.09565090001507E-15"
+        ixz="-7.90343014493262E-08"
         iyy="2.29560460356564E-05"
-        iyz="-3.24413152930276E-15"
+        iyz="-3.24413089402805E-15"
         izz="2.33418727819674E-05" />
     </inertial>
@@ -412,5 +418,5 @@
     <inertial>
       <origin
-        xyz="1.40778055879309E-10 -0.00351477760970662 -0.00156804367684214"
+        xyz="1.40778055879309E-10 -0.00351477760970662 -0.00156804367684215"
         rpy="0 0 0" />
       <mass
@@ -418,6 +424,6 @@
       <inertia
         ixx="2.29560460356564E-05"
-        ixy="-7.09564727696399E-15"
-        ixz="3.24413364688513E-15"
+        ixy="-7.09564736960822E-15"
+        ixz="3.24413279985218E-15"
         iyy="7.00800168489502E-07"
         iyz="7.90343014493306E-08"

File: robot_da/src/robot_docking/urdf/robot_properties.xacro (robot description, xacro)
@@ -1,10 +1,4 @@
 <?xml version="1.0" encoding="utf-8"?>
 <robot name="robot_docking" xmlns:xacro="http://www.ros.org/wiki/xacro">
-<xacro:property name="base_length" value="0.13" />
-<xacro:property name="base_width" value="0.13" />
-<xacro:property name="base_height" value="0.13" />
-<xacro:property name="wheel_radius" value="02" />
-<xacro:property name="wheel_length" value="0.07" />
-<xacro:property name="wheel_joint_pos" value="0.02" />
 <transmission name="front_wheel_trans">
     <type>transmission_interface/SimpleTransmission</type>
